File: hardware/prep.kicad_sch (KiCad schematic)
At the start: 20 parts, among them U1 LD1117S33TR_SOT223, U2 LM4040DBZ-10

Commit message: More available, cheaper parts & fix BOM (#6)
* Change to voltage ref more available at JLCPCB

* more available, cheaper 10 uF cap

* prepping to make makefile work with multiple sch

* cheaper 100 nF cap

* Generate BOM per sch, then merge

* remove unused VERSIONED_SCHEMATIC

* hide some boring ops

* o ya install rename
Parts:
- C8: LCSC C17314042 -> C17024
- C9: LCSC C7411876 -> C77456
- U2: LCSC C3717582 -> C201738
Changed lines of the file:
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@@
 			)
 		)
-		(property "LCSC" "C3717582"
+		(property "LCSC" "C201738"
 			(at 198.12 119.38 0)
 			(effects
@@
 			)
 		)
-		(property "LCSC" "C17314042"
+		(property "LCSC" "C17024"
 			(at 91.44 144.78 0)
 			(effects
@@
 			)
 		)
-		(property "LCSC" "C7411876"
+		(property "LCSC" "C77456"
 			(at 104.14 144.78 0)
 			(effects
