File: hardware/prep.kicad_sch (KiCad schematic)
At the start: 20 parts, among them U1 LD1117S33TR_SOT223, U2 LM4040DBZ-10

Commit message: Change to voltage ref more available at JLCPCB
Parts:
- U2: LCSC C3717582 -> C201738
Changed lines of the file:
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@@
 			)
 		)
-		(property "LCSC" "C3717582"
+		(property "LCSC" "C201738"
 			(at 198.12 119.38 0)
 			(effects

Commit message: more available, cheaper 10 uF cap
Parts:
- C8: LCSC C17314042 -> C17024
Changed lines of the file:
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@@
 			)
 		)
-		(property "LCSC" "C17314042"
+		(property "LCSC" "C17024"
 			(at 91.44 144.78 0)
 			(effects

Commit message: cheaper 100 nF cap
Parts:
- C9: LCSC C7411876 -> C77456
Changed lines of the file:
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@@
 			)
 		)
-		(property "LCSC" "C7411876"
+		(property "LCSC" "C77456"
 			(at 104.14 144.78 0)
 			(effects

Commit message: Changed 2.2kR resistor to something more available (#7)
Parts:
- R1: LCSC C6549338 -> C284423
Changed lines of the file:
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@@
 			)
 		)
-		(property "LCSC" "C6549338"
+		(property "LCSC" "C284423"
 			(at 186.69 119.38 90)
 			(effects

Commit message: Flipped -12V rail b/c I had it wrong
Connections:
- net -12V: now also D3.2 (A); no longer D3.1 (K)
- net at FB3.2: now also D3.1 (K); no longer D3.2 (A)
Other:
- moved on the sheet: D3
Changed lines of the file:
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@@
 	(symbol
 		(lib_id "Device:D")
-		(at 86.36 69.85 180)
+		(at 86.36 69.85 0)
 		(unit 1)
 		(exclude_from_sim no)
